File: HP6632B_relay_board.kicad_pcb (KiCad board)
At the start: 2 copper layers, 67.1 x 56.6 mm, 23 parts, among them J1 Molex 26-60-4090 (KK396), J610 68610814422 8 pos 1mm FFC, J620 Molex 09-48-1094 or 09-48-3095, K601 V23105-A5303-A201, K602 V23105-A5303-A201, K603 V23105-A5303-A201, K604 ST2-DC12V-F, K605 ST2-DC12V-F, U601 NCV1413B

Commit message: update to newer kicad version, added interactive BOM
Parts:
- F601, F602: value Bussmann SS-5H-1.25A-APH -> 1.25A
- K601, K602, K603: value V23105-A5303-A201 -> Relay DPDT
- K604, K605: value ST2-DC12V-F -> Relay DPST
